File: CM4CB/CM4CB.sch (KiCad schematic (older format))
At the start: 0 parts

Commit message: recreate repo without datasheets
Parts:
- added C?: 10uF, symbol Device:C
- added D?: 1N4148, digikey-footprints:Diode_DO-35_P10mm, symbol dk_Diodes-Rectifiers-Single:1N4148
- added R?: 10K, symbol Device:R
- added U?: KSZ9567S, Package_QFP:TQFP-128_14x14mm_P0.4mm, symbol CM4CB:KSZ9567S
Connections:
- new net: C?.1, D?.2, R?.2, U?.96 (RESET_N)
- new net: D?.1, R?.1
- new net TD1+NET1: U?.1 (TXRX1P_A)
- new net TD1+NET2: U?.12 (TXRX2P_A)
- new net TD1+NET3: U?.24 (TXRX3P_A)
- new net TD1+NET4: U?.34 (TXRX4P_A)
- new net TD1+NET5: U?.112 (TXRX5P_A)
- new net TD1-NET1: U?.2 (TXRX1M_A)
- new net TD1-NET2: U?.13 (TXRX2M_A)
- new net TD1-NET3: U?.25 (TXRX3M_A)
- new net TD1-NET4: U?.35 (TXRX4M_A)
- new net TD1-NET5: U?.113 (TXRX5M_A)
- new net TD2+NET1: U?.4 (TXRX1P_B)
- new net TD2+NET2: U?.15 (TXRX2P_B)
- new net TD2+NET3: U?.26 (TXRX3P_B)
- new net TD2+NET4: U?.37 (TXRX4P_B)
- new net TD2+NET5: U?.115 (TXRX5P_B)
- new net TD2-NET1: U?.5 (TXRX1M_B)
- new net TD2-NET2: U?.16 (TXRX2M_B)
- new net TD2-NET3: U?.27 (TXRX3M_B)
- new net TD2-NET4: U?.38 (TXRX4M_B)
- new net TD2-NET5: U?.116 (TXRX5M_B)
- new net TD3+NET1: U?.6 (TXRX1P_C)
- new net TD3+NET2: U?.17 (TXRX2P_C)
- new net TD3+NET3: U?.28 (TXRX3P_C)
- new net TD3+NET4: U?.39 (TXRX4P_C)
- new net TD3+NET5: U?.117 (TXRX5P_C)
- new net TD3-NET1: U?.7 (TXRX1M_C)
- new net TD3-NET2: U?.18 (TXRX2M_C)
- new net TD3-NET3: U?.29 (TXRX3M_C)
- new net TD3-NET4: U?.40 (TXRX4M_C)
- new net TD3-NET5: U?.118 (TXRX5M_C)
- new net TD4+NET1: U?.8 (TXRX1P_D)
- new net TD4+NET2: U?.20 (TXRX2P_D)
- new net TD4+NET3: U?.31 (TXRX3P_D)
- new net TD4+NET4: U?.42 (TXRX4P_D)
- new net TD4+NET5: U?.120 (TXRX5P_D)
- new net TD4-NET1: U?.9 (TXRX1M_D)
- new net TD4-NET2: U?.21 (TXRX2M_D)
- new net TD4-NET3: U?.32 (TXRX3M_D)
- new net TD4-NET4: U?.43 (TXRX4M_D)
- new net TD4-NET5: U?.121 (TXRX5M_D)
